Commit message: added dual arm SDK hardware interface

File: src/dual_arm_robot/config/dual_arm.ros2_control.xacro (robot description, xacro)
@@ -1,5 +1,5 @@
 <?xml version="1.0"?>
 <robot xmlns:xacro="http://www.ros.org/wiki/xacro">
-  <xacro:macro name="realman_arm_ros2_control" params="sim_left sim_right namespace">
+  <xacro:macro name="realman_arm_ros2_control" params="sim_left sim_right namespace config_prefix">
     <ros2_control name="right_arm" type="system">
       <hardware>
@@ -8,10 +8,12 @@
         </xacro:if>
         <xacro:unless value="${sim_right}">
-          <plugin>realman_arm_hardware_interface/RealmanArmHardwareInterface</plugin>
+          <!-- <plugin>realman_arm_hardware_interface/RealmanRightArmHardwareInterface</plugin> -->
+          <plugin>dual_arm_hardware_interface/RightArmHardwareInterface</plugin>
+          <param name="config_prefix">${config_prefix}</param>
         </xacro:unless>
       </hardware>
       <joint name="arm_J1_r">
         <command_interface name="position"/>
-        <command_interface name="effort"/>
+        <!-- <command_interface name="effort"/> -->
         <state_interface name="position"/>
         <state_interface name="velocity"/>
@@ -19,5 +21,5 @@
       <joint name="arm_J2_r">
         <command_interface name="position"/>
-        <command_interface name="effort"/>
+        <!-- <command_interface name="effort"/> -->
         <state_interface name="position"/>
         <state_interface name="velocity"/>
@@ -25,5 +27,5 @@
       <joint name="arm_J3_r">
         <command_interface name="position"/>
-        <command_interface name="effort"/>
+        <!-- <command_interface name="effort"/> -->
         <state_interface name="position"/>
         <state_interface name="velocity"/>
@@ -31,5 +33,5 @@
       <joint name="arm_J4_r">
         <command_interface name="position"/>
-        <command_interface name="effort"/>
+        <!-- <command_interface name="effort"/> -->
         <state_interface name="position"/>
         <state_interface name="velocity"/>
@@ -37,5 +39,5 @@
       <joint name="arm_J5_r">
         <command_interface name="position"/>
-        <command_interface name="effort"/>
+        <!-- <command_interface name="effort"/> -->
         <state_interface name="position"/>
         <state_interface name="velocity"/>
@@ -43,5 +45,5 @@
       <joint name="arm_J6_r">
         <command_interface name="position"/>
-        <command_interface name="effort"/>
+        <!-- <command_interface name="effort"/> -->
         <state_interface name="position"/>
         <state_interface name="velocity"/>
@@ -49,5 +51,5 @@
       <joint name="arm_J7_r">
         <command_interface name="position"/>
-        <command_interface name="effort"/>
+        <!-- <command_interface name="effort"/> -->
         <state_interface name="position"/>
         <state_interface name="velocity"/>
@@ -60,10 +62,12 @@
         </xacro:if>
         <xacro:unless value="${sim_left}">
-          <plugin>realman_arm_hardware_interface/RealmanArmHardwareInterface</plugin>
+          <!-- <plugin>realman_arm_hardware_interface/RealmanLeftArmHardwareInterface</plugin> -->
+          <plugin>dual_arm_hardware_interface/LeftArmHardwareInterface</plugin>
+          <param name="config_prefix">${config_prefix}</param>
         </xacro:unless>
       </hardware>
         <joint name="arm_J1_l">
           <command_interface name="position"/>
-          <command_interface name="effort"/>
+          <!-- <command_interface name="effort"/> -->
           <state_interface name="position"/>
           <state_interface name="velocity"/>
@@ -71,5 +75,5 @@
         <joint name="arm_J2_l">
           <command_interface name="position"/>
-          <command_interface name="effort"/>
+          <!-- <command_interface name="effort"/> -->
           <state_interface name="position"/>
           <state_interface name="velocity"/>
@@ -77,5 +81,5 @@
         <joint name="arm_J3_l">
           <command_interface name="position"/>
-          <command_interface name="effort"/>
+          <!-- <command_interface name="effort"/> -->
           <state_interface name="position"/>
           <state_interface name="velocity"/>
@@ -83,5 +87,5 @@
         <joint name="arm_J4_l">
           <command_interface name="position"/>
-          <command_interface name="effort"/>
+          <!-- <command_interface name="effort"/> -->
           <state_interface name="position"/>
           <state_interface name="velocity"/>
@@ -89,5 +93,5 @@
         <joint name="arm_J5_l">
           <command_interface name="position"/>
-          <command_interface name="effort"/>
+          <!-- <command_interface name="effort"/> -->
           <state_interface name="position"/>
           <state_interface name="velocity"/>
@@ -95,5 +99,5 @@
         <joint name="arm_J6_l">
           <command_interface name="position"/>
-          <command_interface name="effort"/>
+          <!-- <command_interface name="effort"/> -->
           <state_interface name="position"/>
           <state_interface name="velocity"/>
@@ -101,5 +105,5 @@
         <joint name="arm_J7_l">
           <command_interface name="position"/>
-          <command_interface name="effort"/>
+          <!-- <command_interface name="effort"/> -->
           <state_interface name="position"/>
           <state_interface name="velocity"/>

File: src/dual_arm_robot/config/gripper.ros2_control.xacro (robot description, xacro)
@@ -9,5 +9,8 @@
                 </xacro:if>
                 <xacro:unless value="${is_sim}">
-                    <plugin>your_real_gripper_hardware/GripperHardwareInterface</plugin>
+                    <plugin>dual_arm_hardware_interface/LeftGripperHardwareInterface</plugin>
+                    <param name="config_prefix">$(arg config_prefix)</param>
+                    <param name="gripper_speed">500</param>
+                    <param name="gripper_force">500</param>
                 </xacro:unless>
             </hardware>

File: src/dual_arm_robot/urdf/dual_arm_robot.urdf.xacro (robot description, xacro)
@@ -3,5 +3,7 @@
 	<!-- Declare launch arguments -->
 	<xacro:arg name="left_arm_sim" default="true" />
+	<xacro:arg name="left_gripper_sim" default="true" />
 	<xacro:arg name="right_arm_sim" default="true" />
+	<xacro:arg name="right_gripper_sim" default="true" />
 	<mujoco>
 		<compiler meshdir="meshes/visual/" balanceinertia="true" discardvisual="false" />
@@ -199,5 +201,6 @@
 		sim_left="$(arg left_arm_sim)"
 		sim_right="$(arg right_arm_sim)"
-		namespace="arm" />
+		namespace="arm"
+		config_prefix="$(arg config_prefix)" />
 	<!-- Left Hand -->
 	<joint name="hand_J0_l" type="fixed">
@@ -214,5 +217,5 @@
 	<xacro:inspire_hand_l_ros2_control
 		name="LeftHand"
-		is_sim="$(arg left_arm_sim)" />
+		is_sim="$(arg left_gripper_sim)" />
 	<xacro:inspire_hand_l_macro base_link="hand_base_link_l"
 				meshdir="package://dual_arm_robot/meshes/inspire_hand_l" />
@@ -221,5 +224,5 @@
 		name="RightGripper"
 		prefix="gripper_"
-		is_sim="$(arg right_arm_sim)" />
+		is_sim="$(arg right_gripper_sim)" />
 	<xacro:gripper_macro end_effector_link="arm_end_effector_r" prefix="arm"
 		meshdir="package://dual_arm_robot/meshes/gripper" suffix="r"
