Commit message: backup source code

File: src/dual_arm_robot/config/dual_arm.ros2_control.xacro (robot description, xacro)
@@ -1,19 +1,98 @@
 <?xml version="1.0"?>
 <robot xmlns:xacro="http://www.ros.org/wiki/xacro">
-  <xacro:macro name="realman_arm_ros2_control" params="sim_left sim_right namespace config_prefix">
-    <ros2_control name="right_arm" type="system">
+  <!-- ============================================================
+       Dual-arm (left + right) combined ros2_control block.
+       Why combined:
+         The SDK uses a single 100 Hz UDP command channel. Every
+         ControlApi::move_joint(group, ...) rewrites the JointCmd array
+         for the WHOLE robot, filling non-selected arms with their
+         current feedback. If left and right arms are separate
+         SystemInterface instances, controller_manager calls write()
+         twice per cycle → two UDP packets → rt_control drops one and
+         the other arm gets frozen at its current position.
+         Combining into ONE SystemInterface ensures one packet per cycle
+         containing targets for every joint (left + head + right).
+       Params:
+         sim_left      : "true" / "false" — left arm simulation
+         sim_right     : "true" / "false" — right arm simulation
+         config_prefix : directory containing config.yaml
+         namespace     : optional, kept for compatibility with the
+                         caller's existing macro signature
+       ============================================================ -->
+  <xacro:macro name="realman_arm_ros2_control"
+               params="sim_left sim_right config_prefix namespace:=''">
+    <ros2_control name="dual_arms" type="system">
       <hardware>
-        <xacro:if value="${sim_right}">
-          <plugin>mock_components/GenericSystem</plugin>
-        </xacro:if>
-        <xacro:unless value="${sim_right}">
-          <!-- <plugin>realman_arm_hardware_interface/RealmanRightArmHardwareInterface</plugin> -->
-          <plugin>dual_arm_hardware_interface/RightArmHardwareInterface</plugin>
-          <param name="config_prefix">${config_prefix}</param>
-        </xacro:unless>
-      </hardware>
+      <!-- Both sides simulated → plain mock passthrough -->
+      <xacro:if value="${str(sim_left).lower() == 'true' and str(sim_right).lower() == 'true'}">
+        <plugin>mock_components/GenericSystem</plugin>
+      </xacro:if>
+      <!-- At least one side real → real plugin -->
+      <xacro:unless value="${str(sim_left).lower() == 'true' and str(sim_right).lower() == 'true'}">
+        <plugin>dual_arm_hardware_interface/DualArmsHardwareInterface</plugin>
+        <param name="config_prefix">${config_prefix}</param>
+        <param name="sim_left">${sim_left}</param>
+        <param name="sim_right">${sim_right}</param>
+        <param name="trajectory_mode">2</param>
+        <param name="trajectory_radio">500</param>
+      </xacro:unless>
+    </hardware>
+      <!-- ============================================================
+           Left arm — 7 joints
+           The hardware interface classifies joints by name suffix:
+             *_l → SDK arm[0]  (left)
+             *_r → SDK arm[2]  (right)
+             other → SDK arm[1] (head)
+           ============================================================ -->
+      <joint name="arm_J1_l">
+        <command_interface name="position"/>
+        <state_interface name="position"/>
+        <state_interface name="velocity"/>
+      </joint>
+      <joint name="arm_J2_l">
+        <command_interface name="position"/>
+        <state_interface name="position"/>
+        <state_interface name="velocity"/>
+      </joint>
+      <joint name="arm_J3_l">
+        <command_interface name="position"/>
+        <state_interface name="position"/>
+        <state_interface name="velocity"/>
+      </joint>
+      <joint name="arm_J4_l">
+        <command_interface name="position"/>
+        <state_interface name="position"/>
+        <state_interface name="velocity"/>
+      </joint>
+      <joint name="arm_J5_l">
+        <command_interface name="position"/>
+        <state_interface name="position"/>
+        <state_interface name="velocity"/>
+      </joint>
+      <joint name="arm_J6_l">
+        <command_interface name="position"/>
+        <state_interface name="position"/>
+        <state_interface name="velocity"/>
+      </joint>
+      <joint name="arm_J7_l">
+        <command_interface name="position"/>
+        <state_interface name="position"/>
+        <state_interface name="velocity"/>
+      </joint>
+      <joint name="head_pan">
+        <command_interface name="position"/>
+        <state_interface name="position"/>
+        <state_interface name="velocity"/>
+      </joint>
+      <joint name="head_tilt">
+        <command_interface name="position"/>
+        <state_interface name="position"/>
+        <state_interface name="velocity"/>
+      </joint>
+      <!-- ============================================================
+           Right arm — 7 joints
+           ============================================================ -->
       <joint name="arm_J1_r">
         <command_interface name="position"/>
-        <!-- <command_interface name="effort"/> -->
         <state_interface name="position"/>
         <state_interface name="velocity"/>
@@ -21,5 +100,4 @@
       <joint name="arm_J2_r">
         <command_interface name="position"/>
-        <!-- <command_interface name="effort"/> -->
         <state_interface name="position"/>
         <state_interface name="velocity"/>
@@ -27,5 +105,4 @@
       <joint name="arm_J3_r">
         <command_interface name="position"/>
-        <!-- <command_interface name="effort"/> -->
         <state_interface name="position"/>
         <state_interface name="velocity"/>
@@ -33,5 +110,4 @@
       <joint name="arm_J4_r">
         <command_interface name="position"/>
-        <!-- <command_interface name="effort"/> -->
         <state_interface name="position"/>
         <state_interface name="velocity"/>
@@ -39,5 +115,4 @@
       <joint name="arm_J5_r">
         <command_interface name="position"/>
-        <!-- <command_interface name="effort"/> -->
         <state_interface name="position"/>
         <state_interface name="velocity"/>
@@ -45,5 +120,4 @@
       <joint name="arm_J6_r">
         <command_interface name="position"/>
-        <!-- <command_interface name="effort"/> -->
         <state_interface name="position"/>
         <state_interface name="velocity"/>
@@ -51,63 +125,8 @@
       <joint name="arm_J7_r">
         <command_interface name="position"/>
-        <!-- <command_interface name="effort"/> -->
         <state_interface name="position"/>
         <state_interface name="velocity"/>
       </joint>
     </ros2_control>
-    <ros2_control name="left_arm" type="system">
-      <hardware>
-        <xacro:if value="${sim_left}">
-          <plugin>mock_components/GenericSystem</plugin>
-        </xacro:if>
-        <xacro:unless value="${sim_left}">
-          <!-- <plugin>realman_arm_hardware_interface/RealmanLeftArmHardwareInterface</plugin> -->
-          <plugin>dual_arm_hardware_interface/LeftArmHardwareInterface</plugin>
-          <param name="config_prefix">${config_prefix}</param>
-        </xacro:unless>
-      </hardware>
-        <joint name="arm_J1_l">
-          <command_interface name="position"/>
-          <!-- <command_interface name="effort"/> -->
-          <state_interface name="position"/>
-          <state_interface name="velocity"/>
-        </joint>
-        <joint name="arm_J2_l">
-          <command_interface name="position"/>
-          <!-- <command_interface name="effort"/> -->
-          <state_interface name="position"/>
-          <state_interface name="velocity"/>
-        </joint>
-        <joint name="arm_J3_l">
-          <command_interface name="position"/>
-          <!-- <command_interface name="effort"/> -->
-          <state_interface name="position"/>
-          <state_interface name="velocity"/>
-        </joint>
-        <joint name="arm_J4_l">
-          <command_interface name="position"/>
-          <!-- <command_interface name="effort"/> -->
-          <state_interface name="position"/>
-          <state_interface name="velocity"/>
-        </joint>
-        <joint name="arm_J5_l">
-          <command_interface name="position"/>
-          <!-- <command_interface name="effort"/> -->
-          <state_interface name="position"/>
-          <state_interface name="velocity"/>
-        </joint>
-        <joint name="arm_J6_l">
-          <command_interface name="position"/>
-          <!-- <command_interface name="effort"/> -->
-          <state_interface name="position"/>
-          <state_interface name="velocity"/>
-        </joint>
-        <joint name="arm_J7_l">
-          <command_interface name="position"/>
-          <!-- <command_interface name="effort"/> -->
-          <state_interface name="position"/>
-          <state_interface name="velocity"/>
-        </joint>
-    </ros2_control>
   </xacro:macro>
 </robot>

File: src/dual_arm_robot/urdf/components/arm_left.urdf.xacro (robot description, xacro)
@@ -272,5 +272,5 @@
 			<parent link="${prefix}_L6_${suffix}" />
 			<child link="${prefix}_L7_${suffix}" />
-			<axis xyz="0 0 1" />
+			<axis xyz="0 0 -1" />
 			<limit effort="0" velocity="5.0" lower="-1.22173" upper="1.22173" />
 		</joint>

File: src/dual_arm_robot/urdf/components/arm_right.urdf.xacro (robot description, xacro)
@@ -222,5 +222,5 @@
 			<parent link="${prefix}_L5_${suffix}" />
 			<child link="${prefix}_L6_${suffix}" />
-			<axis xyz="0 0 1" />
+			<axis xyz="0 0 -1" />
 			<limit effort="0" velocity="5.0" lower="-1.22173" upper="1.22173" />
 		</joint>
@@ -258,5 +258,5 @@
 			<parent link="${prefix}_L6_${suffix}" />
 			<child link="${prefix}_L7_${suffix}" />
-			<axis xyz="0 0 1" />
+			<axis xyz="0 0 -1" />
 			<limit effort="0" velocity="5.0" lower="-1.22173" upper="1.22173" />
 		</joint>

File: src/dual_arm_robot/urdf/dual_arm_robot.urdf.xacro (robot description, xacro)
@@ -173,7 +173,7 @@
 	<xacro:arm_left_macro base_link="base_link" end_effector_link="end_effector" prefix="arm"
 		suffix="l" meshdir="package://dual_arm_robot/meshes/arm"
-		origin_roll="-1.57079632, -1.57079632, 1.57079632 , -1.57079632, 1.57079632, -1.57079632, 1.57079632"
-		origin_pitch="0.000000000, 0.000000000, 0.000000000, 0.000000000, 0.000000000, -1.57079632, 0.000000000"
-		origin_yaw="0.000000000, 0.000000000, 0.000000000, 0.000000000, 0.000000000, 0.000000000, 0.000000000"
+		origin_roll="0.0, -1.57079632, 1.57079632 , -1.57079632, 1.57079632, -1.57079632, 1.57079632"
+		origin_pitch="1.57079632, 0.000000000, 0.000000000, 0.000000000, 0.000000000, -1.57079632, 0.000000000"
+		origin_yaw="1.57079632, 0.000000000, 0.000000000, 0.000000000, 0.000000000, 0.000000000, 0.000000000"
 		origin_x="0.000000000, 0.000000000, 0.000000000, 0.039      , 0.000000000, 0.000000000, 0.067      "
 		origin_y="0.209      , 0.000000000, -0.310      , 0.000000000, -0.310      , 0.000000000, 0.000000000"
@@ -187,7 +187,7 @@
 	<xacro:arm_right_macro base_link="base_link" end_effector_link="end_effector" prefix="arm"
 		suffix="r" meshdir="package://dual_arm_robot/meshes/arm"
-		origin_roll="-1.57079632, 1.57079632 , -1.57079632, 1.57079632, -1.57079632 , 1.57079632 , -1.57079632"
-		origin_pitch="0.000000000, 0.000000000, 0.000000000, 0.000000000, 0.000000000, 1.57079632 , 0.000000000"
-		origin_yaw="0.000000000, 0.000000000, 0.000000000, 0.000000000, 0.000000000, 0.000000000, 0.000000000"
+		origin_roll="0.0, 1.57079632 , -1.57079632, 1.57079632, -1.57079632 , 1.57079632 , -1.57079632"
+		origin_pitch="1.57079632, 0.000000000, 0.000000000, 0.000000000, 0.000000000, 1.57079632 , 0.000000000"
+		origin_yaw="1.57079632, 0.000000000, 0.000000000, 0.000000000, 0.000000000, 0.000000000, 0.000000000"
 		origin_x="0.000000000, 0.000000000, 0.000000000, 0.039      , 0.000000000, 0.000000000, 0.067      "
 		origin_y="-0.209     , 0.000000000, -0.310      , 0.000000000, -0.310      , 0.000000000, 0.000000000"
@@ -234,3 +234,30 @@
 	</joint>
 	<link name="tcp_r"/>
+	<link name="head_pan_link"/>
+    <joint name="head_pan" type="revolute">
+      <parent link="arm_base_link_l"/>
+      <child  link="head_pan_link"/>
+      <origin xyz="0 0 1.2" rpy="0 0 0"/>   <!-- 改：头部安装位置 -->
+      <axis   xyz="0 0 1"/>                 <!-- 绕 Z 轴旋转 -->
+      <limit  lower="-3.14" upper="3.14"
+              effort="10.0" velocity="1.5"/>
+    </joint>
+    <!-- ============================================ -->
+    <!-- Tilt joint: pitch rotation (around Y)        -->
+    <!-- ============================================ -->
+    <link name="head_tilt_link"/>
+    <joint name="head_tilt" type="revolute">
+      <parent link="head_pan_link"/>
+      <child  link="head_tilt_link"/>
+      <origin xyz="0 0 0" rpy="0 0 0"/>
+      <axis   xyz="0 1 0"/>
+      <limit  lower="-0.5" upper="0.5"
+              effort="5.0" velocity="1.0"/>
+    </joint>
+    <link name="head_camera_link"/>
+    <joint name="head_camera_joint" type="fixed">
+      <parent link="head_tilt_link"/>
+      <child  link="head_camera_link"/>
+      <origin xyz="0.08 0 0" rpy="0 0 0"/>
+    </joint>
 </robot>

File: src/xr_bringup/config/dual_arm.ros2_control.xacro (robot description, xacro)
@@ -1,17 +1,87 @@
 <?xml version="1.0"?>
 <robot xmlns:xacro="http://www.ros.org/wiki/xacro">
-  <xacro:macro name="realman_arm_ros2_control" params="sim_left sim_right namespace">
-    <ros2_control name="right_arm" type="system">
+  <!-- ============================================================
+       Dual-arm (left + right) combined ros2_control block.
+       Why combined:
+         The SDK uses a single 100 Hz UDP command channel. Every
+         ControlApi::move_joint(group, ...) rewrites the JointCmd array
+         for the WHOLE robot, filling non-selected arms with their
+         current feedback. If left and right arms are separate
+         SystemInterface instances, controller_manager calls write()
+         twice per cycle → two UDP packets → rt_control drops one and
+         the other arm gets frozen at its current position.
+         Combining into ONE SystemInterface ensures one packet per cycle
+         containing targets for every joint (left + head + right).
+       Params:
+         sim_left      : "true" / "false" — left arm simulation
+         sim_right     : "true" / "false" — right arm simulation
+         config_prefix : directory containing config.yaml
+         namespace     : optional, kept for compatibility with the
+                         caller's existing macro signature
+       ============================================================ -->
+  <xacro:macro name="realman_arm_ros2_control"
+               params="sim_left sim_right config_prefix namespace:=''">
+    <ros2_control name="dual_arms" type="system">
       <hardware>
-        <xacro:if value="${sim_right}">
+        <!-- Both sides simulated → plain mock passthrough -->
+        <xacro:if value="${sim_left == 'true' and sim_right == 'true'}">
           <plugin>mock_components/GenericSystem</plugin>
         </xacro:if>
-        <xacro:unless value="${sim_right}">
-          <plugin>realman_arm_hardware_interface/RealmanArmHardwareInterface</plugin>
+        <!-- At least one side real → real plugin; the flags tell the
+             hardware interface which side to hold at feedback position -->
+        <xacro:unless value="${sim_left == 'true' and sim_right == 'true'}">
+          <plugin>dual_arm_hardware_interface/DualArmsHardwareInterface</plugin>
+          <param name="config_prefix">${config_prefix}</param>
+          <param name="sim_left">${sim_left}</param>
+          <param name="sim_right">${sim_right}</param>
         </xacro:unless>
       </hardware>
+      <!-- ============================================================
+           Left arm — 7 joints
+           The hardware interface classifies joints by name suffix:
+             *_l → SDK arm[0]  (left)
+             *_r → SDK arm[2]  (right)
+             other → SDK arm[1] (head)
+           ============================================================ -->
+      <joint name="arm_J1_l">
+        <command_interface name="position"/>
+        <state_interface name="position"/>
+        <state_interface name="velocity"/>
+      </joint>
+      <joint name="arm_J2_l">
+        <command_interface name="position"/>
+        <state_interface name="position"/>
+        <state_interface name="velocity"/>
+      </joint>
+      <joint name="arm_J3_l">
+        <command_interface name="position"/>
+        <state_interface name="position"/>
+        <state_interface name="velocity"/>
+      </joint>
+      <joint name="arm_J4_l">
+        <command_interface name="position"/>
+        <state_interface name="position"/>
+        <state_interface name="velocity"/>
+      </joint>
+      <joint name="arm_J5_l">
+        <command_interface name="position"/>
+        <state_interface name="position"/>
+        <state_interface name="velocity"/>
+      </joint>
+      <joint name="arm_J6_l">
+        <command_interface name="position"/>
+        <state_interface name="position"/>
+        <state_interface name="velocity"/>
+      </joint>
+      <joint name="arm_J7_l">
+        <command_interface name="position"/>
+        <state_interface name="position"/>
+        <state_interface name="velocity"/>
+      </joint>
+      <!-- ============================================================
+           Right arm — 7 joints
+           ============================================================ -->
       <joint name="arm_J1_r">
         <command_interface name="position"/>
-        <command_interface name="effort"/>
         <state_interface name="position"/>
         <state_interface name="velocity"/>
@@ -19,5 +89,4 @@
       <joint name="arm_J2_r">
         <command_interface name="position"/>
-        <command_interface name="effort"/>
         <state_interface name="position"/>
         <state_interface name="velocity"/>
@@ -25,5 +94,4 @@
       <joint name="arm_J3_r">
         <command_interface name="position"/>
-        <command_interface name="effort"/>
         <state_interface name="position"/>
         <state_interface name="velocity"/>
@@ -31,5 +99,4 @@
       <joint name="arm_J4_r">
         <command_interface name="position"/>
-        <command_interface name="effort"/>
         <state_interface name="position"/>
         <state_interface name="velocity"/>
@@ -37,5 +104,4 @@
       <joint name="arm_J5_r">
         <command_interface name="position"/>
-        <command_interface name="effort"/>
         <state_interface name="position"/>
         <state_interface name="velocity"/>
@@ -43,5 +109,4 @@
       <joint name="arm_J6_r">
         <command_interface name="position"/>
-        <command_interface name="effort"/>
         <state_interface name="position"/>
         <state_interface name="velocity"/>
@@ -49,61 +114,19 @@
       <joint name="arm_J7_r">
         <command_interface name="position"/>
-        <command_interface name="effort"/>
+        <state_interface name="position"/>
+        <state_interface name="velocity"/>
+      </joint>
+      <!-- If you ever add a head, declare it here without a suffix, e.g.: -->
+      <joint name="head_pan">
+        <command_interface name="position"/>
+        <state_interface name="position"/>
+        <state_interface name="velocity"/>
+      </joint>
+      <joint name="head_tilt">
+        <command_interface name="position"/>
         <state_interface name="position"/>
         <state_interface name="velocity"/>
       </joint>
     </ros2_control>
-    <ros2_control name="left_arm" type="system">
-      <hardware>
-        <xacro:if value="${sim_left}">
-          <plugin>mock_components/GenericSystem</plugin>
-        </xacro:if>
-        <xacro:unless value="${sim_left}">
-          <plugin>realman_arm_hardware_interface/RealmanArmHardwareInterface</plugin>
-        </xacro:unless>
-      </hardware>
-        <joint name="arm_J1_l">
-          <command_interface name="position"/>
-          <command_interface name="effort"/>
-          <state_interface name="position"/>
-          <state_interface name="velocity"/>
-        </joint>
-        <joint name="arm_J2_l">
-          <command_interface name="position"/>
-          <command_interface name="effort"/>
-          <state_interface name="position"/>
-          <state_interface name="velocity"/>
-        </joint>
-        <joint name="arm_J3_l">
-          <command_interface name="position"/>
-          <command_interface name="effort"/>
-          <state_interface name="position"/>
-          <state_interface name="velocity"/>
-        </joint>
-        <joint name="arm_J4_l">
-          <command_interface name="position"/>
-          <command_interface name="effort"/>
-          <state_interface name="position"/>
-          <state_interface name="velocity"/>
-        </joint>
-        <joint name="arm_J5_l">
-          <command_interface name="position"/>
-          <command_interface name="effort"/>
-          <state_interface name="position"/>
-          <state_interface name="velocity"/>
-        </joint>
-        <joint name="arm_J6_l">
-          <command_interface name="position"/>
-          <command_interface name="effort"/>
-          <state_interface name="position"/>
-          <state_interface name="velocity"/>
-        </joint>
-        <joint name="arm_J7_l">
-          <command_interface name="position"/>
-          <command_interface name="effort"/>
-          <state_interface name="position"/>
-          <state_interface name="velocity"/>
-        </joint>
-    </ros2_control>
   </xacro:macro>
 </robot>
