Commit message: backup source code

File: src/dual_arm_robot/urdf/components/arm_left.urdf.xacro (robot description, xacro)
@@ -272,5 +272,5 @@
 			<parent link="${prefix}_L6_${suffix}" />
 			<child link="${prefix}_L7_${suffix}" />
-			<axis xyz="0 0 -1" />
+			<axis xyz="0 0 1" />
 			<limit effort="0" velocity="5.0" lower="-1.22173" upper="1.22173" />
 		</joint>

File: src/dual_arm_robot/urdf/components/arm_right.urdf.xacro (robot description, xacro)
@@ -222,5 +222,5 @@
 			<parent link="${prefix}_L5_${suffix}" />
 			<child link="${prefix}_L6_${suffix}" />
-			<axis xyz="0 0 -1" />
+			<axis xyz="0 0 1" />
 			<limit effort="0" velocity="5.0" lower="-1.22173" upper="1.22173" />
 		</joint>
@@ -258,5 +258,5 @@
 			<parent link="${prefix}_L6_${suffix}" />
 			<child link="${prefix}_L7_${suffix}" />
-			<axis xyz="0 0 -1" />
+			<axis xyz="0 0 1" />
 			<limit effort="0" velocity="5.0" lower="-1.22173" upper="1.22173" />
 		</joint>

File: src/dual_arm_robot/urdf/dual_arm_robot.urdf.xacro (robot description, xacro)
@@ -173,7 +173,7 @@
 	<xacro:arm_left_macro base_link="base_link" end_effector_link="end_effector" prefix="arm"
 		suffix="l" meshdir="package://dual_arm_robot/meshes/arm"
-		origin_roll="0.0, -1.57079632, 1.57079632 , -1.57079632, 1.57079632, -1.57079632, 1.57079632"
-		origin_pitch="1.57079632, 0.000000000, 0.000000000, 0.000000000, 0.000000000, -1.57079632, 0.000000000"
-		origin_yaw="1.57079632, 0.000000000, 0.000000000, 0.000000000, 0.000000000, 0.000000000, 0.000000000"
+		origin_roll="-1.57079632, -1.57079632, 1.57079632 , -1.57079632, 1.57079632, -1.57079632, 1.57079632"
+		origin_pitch="0.000000000, 0.000000000, 0.000000000, 0.000000000, 0.000000000, -1.57079632, 0.000000000"
+		origin_yaw="0.000000000, 0.000000000, 0.000000000, 0.000000000, 0.000000000, 0.000000000, 0.000000000"
 		origin_x="0.000000000, 0.000000000, 0.000000000, 0.039      , 0.000000000, 0.000000000, 0.067      "
 		origin_y="0.209      , 0.000000000, -0.310      , 0.000000000, -0.310      , 0.000000000, 0.000000000"
@@ -187,7 +187,7 @@
 	<xacro:arm_right_macro base_link="base_link" end_effector_link="end_effector" prefix="arm"
 		suffix="r" meshdir="package://dual_arm_robot/meshes/arm"
-		origin_roll="0.0, 1.57079632 , -1.57079632, 1.57079632, -1.57079632 , 1.57079632 , -1.57079632"
-		origin_pitch="1.57079632, 0.000000000, 0.000000000, 0.000000000, 0.000000000, 1.57079632 , 0.000000000"
-		origin_yaw="1.57079632, 0.000000000, 0.000000000, 0.000000000, 0.000000000, 0.000000000, 0.000000000"
+		origin_roll="-1.57079632, 1.57079632 , -1.57079632, 1.57079632, -1.57079632 , 1.57079632 , -1.57079632"
+		origin_pitch="0.000000000, 0.000000000, 0.000000000, 0.000000000, 0.000000000, 1.57079632 , 0.000000000"
+		origin_yaw="0.000000000, 0.000000000, 0.000000000, 0.000000000, 0.000000000, 0.000000000, 0.000000000"
 		origin_x="0.000000000, 0.000000000, 0.000000000, 0.039      , 0.000000000, 0.000000000, 0.067      "
 		origin_y="-0.209     , 0.000000000, -0.310      , 0.000000000, -0.310      , 0.000000000, 0.000000000"
